File: hardware/asymmetria.kicad_pcb (KiCad board)
At the start: 2 copper layers, 50 x 47 mm, 36 parts, among them P1 CONN_01X02, P2 CONN_01X03, P3 CONN_01X02, P5 CONN_01X02, SW1 3x6x2.5mm, SW2 3x6x2.5mm, U1 AMS1117-3.3, U2 PT4115B89E, U3 ESP8266EX, U4 W25Q32FV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

Commit message: component checks
Parts:
- added W1: MH, Connect:1pin, F.Cu at (127.1, 71.8)
- added W2: MH, Connect:1pin, F.Cu at (151.6, 71.8)
- SW1, SW2: footprint Buttons_Switches_SMD:SW_SPST_EVQPE1 -> umetronics:SPST_3x6x2.5_SMD
- moved SW1 2.17 mm to (121.2, 85.9)
- moved R1 1.27 mm to (122.2, 79.7)
- moved R2 1.27 mm to (120.1, 79.7)
- moved SW2 0.72 mm to (121.2, 95.7), turned to 270 degrees
- moved ANT1 0.06 mm to (126.0, 55.7)
Connections:
- ANT1 pad 2: GND -> (no net)
- U3 pad 33: GND -> (no net)
Routing:
- net GND: track 81.6 -> 230.1 mm, vias 45 -> 98
- net (no net): track 109.7 -> 1.20 mm, vias 53 -> 0
- net /U1_PIN4: track 14.1 -> 28.3 mm, vias 10 -> 20
- net /RESET: track 48.3 -> 54.2 mm
- net +3V3: track 141.6 -> 138.2 mm
- net /GPIO0: track 20.5 -> 17.9 mm
Other:
- rule pad_to_mask_clearance: 0.0508 -> 0.1524
- board text added: "CC BY 4.0 12/2015 aon@umetronics.com"
- board text removed: "CC BY 4.0 11/2015 aon@umetronics.com"
