File: hardware/asymmetria.kicad_pcb (KiCad board)
At the start: 2 copper layers, 50 x 47 mm, 38 parts, among them P1 CONN_01X02, P2 CONN_01X03, P3 CONN_01X02, P5 CONN_01X02, SW1 3x6x2.5mm, SW2 3x6x2.5mm, U1 AMS1117-3.3, U2 PT4115B89E, U3 ESP8266EX, U4 W25Q32FV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

Commit message: grounded qfn center pad, increased C7 to 100uF
Parts:
- C7: value 10uF -> 100uF
- R5, R6: value R -> 4K7
Connections:
- U3 pad 33: (no net) -> GND
Routing:
- net GND: track 230.1 -> 232.6 mm, vias 98 -> 100
Other:
- board text added: "asymmetria-v1.1"
- board text removed: "asymmetria-v1.0"
Changed lines of the file:
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@@
-(kicad_pcb (version 4) (host pcbnew 4.0.0-2.201511301921+6191~38~ubuntu15.10.1-stable)
+(kicad_pcb (version 4) (host pcbnew 4.0.0-2.201512062335+6193~38~ubuntu15.10.1-stable)
   (general
-    (links 87)
-    (no_connects 0)
+    (links 92)
+    (no_connects 1)
     (area 104.924999 53.301899 231.401102 102.075001)
     (thickness 1.6)
     (drawings 11)
-    (tracks 645)
+    (tracks 651)
     (zones 0)
     (modules 38)
@@
     (mod_text_size 1 1)
     (mod_text_width 0.15)
-    (pad_size 1.725 1.725)
+    (pad_size 0.46 0.8)
     (pad_drill 0)
     (pad_to_mask_clearance 0.1524)
@@
       (effects (font (size 1 1) (thickness 0.15)))
     )
-    (fp_text value 10uF (at 0 2.3 180) (layer F.Fab)
+    (fp_text value 100uF (at 0 2.3 180) (layer F.Fab)
       (effects (font (size 1 1) (thickness 0.15)))
     )
@@
       (net 15 /RESET))
     (pad 33 smd rect (at 0.8625 0.8625 270) (size 1.725 1.725) (layers F.Cu F.Paste F.Mask)
-      (solder_paste_margin_ratio -0.2))
+      (net 1 GND) (solder_paste_margin_ratio -0.2))
     (pad 33 smd rect (at 0.8625 -0.8625 270) (size 1.725 1.725) (layers F.Cu F.Paste F.Mask)
-      (solder_paste_margin_ratio -0.2))
+      (net 1 GND) (solder_paste_margin_ratio -0.2))
     (pad 33 smd rect (at -0.8625 0.8625 270) (size 1.725 1.725) (layers F.Cu F.Paste F.Mask)
-      (solder_paste_margin_ratio -0.2))
+      (net 1 GND) (solder_paste_margin_ratio -0.2))
     (pad 33 smd rect (at -0.8625 -0.8625 270) (size 1.725 1.725) (layers F.Cu F.Paste F.Mask)
-      (solder_paste_margin_ratio -0.2))
+      (net 1 GND) (solder_paste_margin_ratio -0.2))
     (model Housings_DFN_QFN.3dshapes/QFN-32-1EP_5x5mm_Pitch0.5mm.wrl
       (at (xyz 0 0 0))
@@
       (effects (font (size 1 1) (thickness 0.15)))
     )
-    (fp_text value R (at 0 1.9 180) (layer F.Fab)
+    (fp_text value 4K7 (at 0 1.9 180) (layer F.Fab)
       (effects (font (size 1 1) (thickness 0.15)))
     )
@@
       (effects (font (size 1 1) (thickness 0.15)))
     )
-    (fp_text value R (at 0 1.9 180) (layer F.Fab)
+    (fp_text value 4K7 (at 0 1.9 180) (layer F.Fab)
       (effects (font (size 1 1) (thickness 0.15)))
     )
@@
       (net 15 /RESET))
   )
-  (gr_text asymmetria-v1.0 (at 158.0515 61.3035) (layer F.SilkS)
+  (gr_text asymmetria-v1.1 (at 158.0515 61.3035) (layer F.SilkS)
     (effects (font (size 0.8 0.8) (thickness 0.15)))
   )
@@
   (segment (start 229.2935 60.0125) (end 229.2935 60.6935) (width 0.1524) (layer F.Cu) (net 0))
   (segment (start 231.0885 60.6935) (end 231.1725 60.6095) (width 0.1524) (layer F.Cu) (net 0) (status 30))
+  (segment (start 136.514 71.925) (end 136.514 71.916) (width 0.1524) (layer F.Cu) (net 1))
+  (segment (start 136.514 71.925) (end 136.5275 71.9385) (width 0.1524) (layer F.Cu) (net 1))
+  (via (at 136.5275 71.9385) (size 0.7112) (drill 0.3556) (layers F.Cu B.Cu) (net 1))
+  (segment (start 136.5275 71.9295) (end 136.5275 71.9385) (width 0.1524) (layer B.Cu) (net 1))
+  (segment (start 136.5275 71.9295) (end 134.789 70.191) (width 0.1524) (layer B.Cu) (net 1))
+  (via (at 134.789 70.191) (size 0.7112) (drill 0.3556) (layers F.Cu B.Cu) (net 1))
   (segment (start 141.224 79.248) (end 141.224 80.731) (width 0.254) (layer B.Cu) (net 1))
   (via (at 139.8515 83.7035) (size 0.7112) (drill 0.3556) (layers F.Cu B.Cu) (net 1))
